Commit message: adding poles.world

File: install/climbbot3_description/share/climbbot3_description/climbbot3/robot.urdf (robot description, URDF)
Before this commit: robot climbbot3, 17 links, 16 joints
Links:
- link assembly_10: mass 0.31630258043837466975 -> 0.316303; geometry collision mesh filename=package://climbbot3_description/climbbot3/assets/part_17.stl; collision mesh filename=package://climbbot3_description/climbbot3/assets/part_22.stl
- link assembly_11: mass 0.23426959223082960415 -> 0.156296; geometry collision mesh filename=package://climbbot3_description/climbbot3/assets/gripper_ho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; collision mesh filename=package://climbbot3_description/climbbot3/assets/part_6.stl
- link assembly_12: mass 0.23426959223082960415 -> 0.156296; geometry collision mesh filename=package://climbbot3_description/climbbot3/assets/gripper_ho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; collision mesh filename=package://climbbot3_description/climbbot3/assets/part_6.stl
- link assembly_13: mass 0.31630263661656304874 -> 0.316303; geometry collision mesh filename=package://climbbot3_description/climbbot3/assets/part_17.stl; collision mesh filename=package://climbbot3_description/climbbot3/assets/part_20.stl
- link assembly_7: mass 0.23604354426025414559 -> 0.236044; geometry collision mesh filename=package://climbbot3_description/climbbot3/assets/component2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; collision mesh filename=package://climbbot3_description/climbbot3/assets/component2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
- link assembly_8: mass 0.11732144979288477993 -> 0.117321; geometry collision mesh filename=package://climbbot3_description/climbbot3/assets/ds3225mg_s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; collision mesh filename=package://climbbot3_description/climbbot3/assets/ds3225mg_s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
- link assembly_9: mass 0.11732144979288477993 -> 0.117321; geometry collision mesh filename=package://climbbot3_description/climbbot3/assets/ds3225mg_s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; collision mesh filename=package://climbbot3_description/climbbot3/assets/ds3225mg_s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
- link part_1: mass 0.14727877470824324302 -> 0.147279; geometry collision mesh filename=package://climbbot3_description/climbbot3/assets/part_1.stl; visual mesh filename=package://climbbot3_description/climbbot3/assets/part_1.stl
- link part_1_2: mass 0.14727877470824324302 -> 0.147279; geometry collision mesh filename=package://climbbot3_description/climbbot3/assets/part_1.stl; visual mesh filename=package://climbbot3_description/climbbot3/assets/part_1.stl
- link part_4: mass 0.11176680215091941428 -> 0.111767; geometry collision mesh filename=package://climbbot3_description/climbbot3/assets/part_4.stl; visual mesh filename=package://climbbot3_description/climbbot3/assets/part_4.stl
- link part_4_2: mass 0.11176680215091941428 -> 0.111767; geometry collision mesh filename=package://climbbot3_description/climbbot3/assets/part_4.stl; visual mesh filename=package://climbbot3_description/climbbot3/assets/part_4.stl
Joints:
- joint l1: limit lower=-1.570796326794896558 upper=1.570796326794896558 effort=100 velocity=20 -> lower=-1.5708 upper=1.5708 effort=1000 velocity=10; origin xyz=0.18085273176231164705 0.019157849104760489578 0.028677557350689036192 rpy=-7.2164496600701612993e-15 -7.1552173200943249137e-15 6.7910954637577480315e-14 -> xyz=0.180853 0.0191578 0.0286776 rpy=1.50377e-30 5.32967e-18 4.55474e-14
- joint l2: limit lower=-1.570796326794896558 upper=1.570796326794896558 effort=100 velocity=20 -> lower=-1.5708 upper=1.5708 effort=1000 velocity=10; origin xyz=0.00056249999998750355168 -0.059799999999987626942 -0.032300000000000390898 rpy=-1.570796326794572817 1.5707963267948663599 0 -> xyz=0.0005625 -0.0598 -0.0323 rpy=-1.5708 1.5708 0
- joint l3_1: limit lower=-0.005 upper=0.13200000000000000622 effort=100 velocity=20 -> lower=-0.007 upper=0.132 effort=1000 velocity=10; origin xyz=0.035000000000058303917 -0.17449999999999193934 -0.031709999999937635295 rpy=1.5707963267951410291 -1.5707963267945699304 0 -> xyz=0.035 -0.1745 -0.03171 rpy=1.5708 -1.5708 0
- joint l3_2: limit lower=-0.005 upper=0.13200000000000000622 effort=100 velocity=20 -> lower=-0.005 upper=0.134 effort=1000 velocity=10; mimic joint=l3_1 multiplier=1.0 offset=0.0 -> joint=l3_1 multiplier=1.0 offset=0.00201; origin xyz=9.7144514654701197287e-17 0 -2.0539125955565395998e-15 rpy=-7.4940054162850202012e-15 -8.4932061383676169492e-15 -7.327471960432721335e-15 -> xyz=7.21645e-16 0 2.55351e-15 rpy=-1.58419e-27 -9.21485e-15 1.38143e-15
- joint l3_3: limit lower=-0.005 upper=0.13400000000000000799 effort=100 velocity=20 -> lower=-0.005 upper=0.134 effort=1000 velocity=10; origin xyz=-6.9388939039072283776e-17 -6.9388939039072283776e-18 0.002000000000013435475 rpy=1.6653345365999751394e-16 3.5363473088349697426e-16 1.6018215753189618816e-16 -> xyz=-7.07767e-16 -6.93889e-18 0.002 rpy=1.4988e-15 4.4964e-15 1.4988e-15
- joint r1: limit lower=-1.570796326794896558 upper=1.570796326794896558 effort=100 velocity=20 -> lower=-1.5708 upper=1.5708 effort=1000 velocity=10; origin xyz=0.18085273176231164705 0.11919956669056486209 0.028677557350689036192 rpy=-6.1232339957420538691e-17 7.1870441298269152156e-28 -6.3108872417680944433e-29 -> xyz=0.180853 0.1192 0.0286776 rpy=-5.78703e-29 5.42099e-27 -5.24704e-14
- joint r2: limit lower=-1.570796326794896558 upper=1.570796326794896558 effort=100 velocity=20 -> lower=-1.5708 upper=1.5708 effort=1000 velocity=10; origin xyz=-0.00056250000000024336089 0.059800000000004821521 -0.032300000000002160316 rpy=1.5707963267948827912 -1.5707963267947857577 0 -> xyz=-0.0005625 0.0598 -0.0323 rpy=1.5708 -1.5708 0
- joint r3_1: limit lower=-0.005 upper=0.13200000000000000622 effort=100 velocity=20 -> lower=-0.007 upper=0.132 effort=1000 velocity=10; origin xyz=-0.035000000000009148793 -0.1744999999999917728 -0.03170999999999701835 rpy=1.570796326794936304 1.57079632679483705 0 -> xyz=-0.035 -0.1745 -0.03171 rpy=1.5708 1.5708 0
- joint r3_2: limit lower=-0.005 upper=0.13200000000000000622 effort=100 velocity=20 -> lower=-0.005 upper=0.134 effort=1000 velocity=10; mimic joint=r3_1 multiplier=1.0 offset=0.0 -> joint=r3_1 multiplier=1.0 offset=0.00201; origin xyz=0 -6.9388939039072283776e-18 6.1062266354383609723e-15 rpy=8.2112531624455133175e-27 -2.2204460492175295007e-16 -2.5243548967072383378e-29 -> xyz=3.05311e-16 0 5.71765e-15 rpy=6.79253e-26 -1.9984e-15 -1.98441e-15
- joint r3_3: limit lower=-0.005 upper=0.13400000000000000799 effort=100 velocity=20 -> lower=-0.005 upper=0.134 effort=1000 velocity=10; origin xyz=2.7755575615628913511e-17 -6.9388939039072283776e-18 0.0020000000000004458656 rpy=6.1232339949145745248e-17 6.1584078566384796889e-16 -2.6015123810540368034e-15 -> xyz=-3.05311e-16 0 0.002 rpy=-4.11758e-30 3.50237e-15 -4.08619e-15
