Commit message: adding simplified gripper

File: src/climbbot3_description/climbbot3/long_gripper_robot.urdf (robot description, URDF)
Before this commit: robot climbbot3, 17 links, 16 joints
Links:
- link assembly_11: mass 0.101166 -> 0.156296; geometry collision mesh filename=package://climbbot3_description/climbbot3/assets/gripper_ho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; collision mesh filename=package://climbbot3_description/climbbot3/assets/part_6.stl
- link assembly_12: mass 0.101166 -> 0.156296; geometry collision mesh filename=package://climbbot3_description/climbbot3/assets/gripper_ho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; collision mesh filename=package://climbbot3_description/climbbot3/assets/part_6.stl
Joints:
- joint l1: origin xyz=0.180853 0.0191578 0.0286776 rpy=1.50377e-30 5.32967e-18 1.92024e-13 -> xyz=0.180853 0.0191578 0.0286776 rpy=1.50377e-30 5.32967e-18 4.55474e-14
- joint l2: limit lower=-1.5708 upper=1.5708 effort=10 velocity=10 -> lower=-1.5708 upper=1.5708 effort=1000 velocity=10
- joint l3_1: limit lower=-0.007 upper=0.132 effort=10 velocity=10 -> lower=-0.007 upper=0.132 effort=1000 velocity=10
- joint l3_2: origin xyz=-1.38778e-17 -1.38778e-17 3.10862e-15 rpy=-5.18013e-28 -1.33227e-15 -3.78022e-27 -> xyz=7.21645e-16 0 2.55351e-15 rpy=-1.58419e-27 -9.21485e-15 1.38143e-15
- joint l3_3: origin xyz=1.38778e-17 6.93889e-18 0.002 rpy=6.12323e-17 -3.66111e-14 3.58539e-14 -> xyz=-7.07767e-16 -6.93889e-18 0.002 rpy=1.4988e-15 4.4964e-15 1.4988e-15
- joint r1: origin xyz=0.180853 0.1192 0.0286776 rpy=8.65347e-17 1.06056e-16 -1.34121e-16 -> xyz=0.180853 0.1192 0.0286776 rpy=-5.78703e-29 5.42099e-27 -5.24704e-14
- joint r3_2: origin xyz=2.22045e-16 0 -2.10942e-15 rpy=6.11244e-25 -1.79856e-14 -7.30202e-17 -> xyz=3.05311e-16 0 5.71765e-15 rpy=6.79253e-26 -1.9984e-15 -1.98441e-15
- joint r3_3: origin xyz=-1.66533e-16 4.85723e-17 0.002 rpy=6.09053e-17 4.63681e-18 7.28027e-17 -> xyz=-3.05311e-16 0 0.002 rpy=-4.11758e-30 3.50237e-15 -4.08619e-15
